Commit message: changed zed_wrapper to current newest zed_wrapper, changed robots file to urdf so arm demo can launch

File: software/ros_packages/zed_wrapper/urdf/include/materials.urdf.xacro (robot description, xacro)
@@ -1,5 +1,5 @@
 <?xml version="1.0"?>
 <!--
-Copyright (c) 2017, STEREOLABS.
+Copyright (c) 2020, STEREOLABS.
 All rights reserved.
 THIS SOFTWARE IS PROVIDED BY THE COPYRIGHT HOLDERS AND CONTRIBUTORS
@@ -15,8 +15,13 @@
 OF THIS SOFTWARE, EVEN IF ADVISED OF THE POSSIBILITY OF SUCH DAMAGE.
 -->
-<launch>
-  <!-- Launch ZED camera wrapper -->
-  <include file="$(find zed_wrapper)/launch/zed.launch" />
-  <!-- Launch rivz display -->
-  <node name="rviz" pkg="rviz" type="rviz" args="-d $(find zed_wrapper)/rviz/zed.rviz" output="screen" />
-</launch>
+<robot>
+    <material name="zed_mat">
+        <color rgba="0.8 0.8 0.8 0.8"/>
+    </material>
+    <material name="zedm_mat">
+        <color rgba="0 0 0 0.9"/>
+    </material>
+    <material name="zed2_mat">
+        <color rgba="0.25 0.25 0.25 0.99"/>
+    </material>
+</robot>
