Commit message: Updated URDF and IKFast Plugin to have correct joint limits

File: software/ros_packages/rover_arm_ik/rover_arm_description/urdf/rover_arm.urdf (robot description, URDF)
Before this commit: robot rover_arm, 8 links, 7 joints
Joints:
- joint base_roll: limit lower=-0.7854 upper=0.7854 effort=150.0 velocity=3.15 -> lower=-3.1415 upper=3.1415 effort=150.0 velocity=3.15
- joint elbow_pitch: limit lower=-1.5708 upper=1.5708 effort=150.0 velocity=3.15 -> lower=-3.1415 upper=3.1415 effort=150.0 velocity=3.15
- joint elbow_roll: limit lower=-1.5708 upper=1.5708 effort=150.0 velocity=3.15 -> lower=-3.1415 upper=3.1415 effort=150.0 velocity=3.15
- joint shoulder_pitch: limit lower=-1.5708 upper=1.5708 effort=150.0 velocity=3.15 -> lower=-3.1415 upper=3.1415 effort=150.0 velocity=3.15
- joint wrist_pitch: limit lower=-1.5708 upper=1.5708 effort=150.0 velocity=3.15 -> lower=-3.1415 upper=3.1415 effort=150.0 velocity=3.15
